File: schematic/heatGun.sch (EAGLE design)
At the start: 36 parts, among them IC1 LD117AS18TR, IC3 STM32F103C8T, IC4 LM358MX, Q2 IRF520, SW1 EC12E_SW, SW2 EC12E_SW, T3 BT138-H

Commit message: Updated schematic
Parts:
- added C2, C4: .1uF, rcl:C-EUC0603
- added C3: 10uF, rcl:CPOL-EUE2,5-6E
- added JP1: (no value), pinhead:PINHD-1X2
- C1: value (none) -> 10uF/35V
- C8: value (none) -> .1uF
- IC1: value LD117AS18TR -> DC-DC converter set to 5v output
Connections:
- net +24V: now also C2.2, IC1.IN
- net +3V3: now also C3.+, C4.2
- net GND: now also C2.1, C3.-, C4.1, JP1.1
- net REED: now also JP1.2
Other:
- moved on the sheet: C1, C12, IC1, IC4A, JP2, JP3, JP6, Q2, R1, R2, R22, R3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
