File: schematic/heatGun.brd (EAGLE design)
At the start: 100 x 80 mm, 36 parts, among them IC1 LD117AS18TR, IC3 STM32F103C8T, IC4 LM358MX, Q2 IRF520, SW1 EC12E_SW, SW2 EC12E_SW, T3 BT138-H

Commit message: Made last settings prevail
Parts:
- added C2, C4: .1uF, rcl:C0603
- added C3: 10uF, rcl:E2,5-6E
- added JP1: (no value), pinhead:1X02
- C1: value (none) -> 10uF/35V
- C8: value (none) -> .1uF
- IC1: value LD117AS18TR -> DC-DC converter set to 5v output
Connections:
- net +24V: now also C2.2, IC1.3
- net +3V3: now also C3.+, C4.2
- net GND: now also C2.1, C3.-, C4.1, JP1.1
- net REED: now also JP1.2
Changed lines of the file:
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@@
 </autorouter>
 <elements>
-<element name="C1" library="rcl" library_urn="urn:adsk.eagle:library:334" package="E2,5-6E" value="" x="-19.05" y="62.23"/>
+<element name="C1" library="rcl" library_urn="urn:adsk.eagle:library:334" package="E2,5-6E" value="10uF/35V" x="-19.05" y="62.23"/>
 <element name="C10" library="rcl" library_urn="urn:adsk.eagle:library:334" package="C0603" value="" x="-16.51" y="85.09"/>
 <element name="C11" library="rcl" library_urn="urn:adsk.eagle:library:334" package="C0603" value="" x="-21.59" y="85.09"/>
 <element name="C12" library="rcl" library_urn="urn:adsk.eagle:library:334" package="C0603" value="" x="-26.67" y="85.09"/>
-<element name="C8" library="rcl" library_urn="urn:adsk.eagle:library:334" package="C0603" value="" x="-45.72" y="85.09"/>
+<element name="C8" library="rcl" library_urn="urn:adsk.eagle:library:334" package="C0603" value=".1uF" x="-45.72" y="85.09"/>
 <element name="D3" library="diode" library_urn="urn:adsk.eagle:library:210" package="F126Z12" value="" x="-26.67" y="67.31"/>
-<element name="IC1" library="v-reg" library_urn="urn:adsk.eagle:library:409" package="SOT223" value="LD117AS18TR" x="-49.53" y="52.07"/>
+<element name="IC1" library="v-reg" library_urn="urn:adsk.eagle:library:409" package="SOT223" value="DC-DC converter set to 5v output" x="-49.53" y="52.07"/>
 <element name="IC3" library="micro-stm_v3" package="LQFP48" value="STM32F103C8T" x="-24.13" y="53.34"/>
 <element name="IC4" library="linear" library_urn="urn:adsk.eagle:library:262" package="SO08" package3d_urn="urn:adsk.eagle:package:16404/2" value="LM358MX" x="-58.42" y="29.21"/>
@@
 <element name="R3" library="rcl" library_urn="urn:adsk.eagle:library:334" package="R0603" value="2K2" x="-69.85" y="-77.47"/>
 <element name="R4" library="rcl" library_urn="urn:adsk.eagle:library:334" package="R0603" value="2K2" x="-64.77" y="-77.47"/>
+<element name="JP1" library="pinhead" library_urn="urn:adsk.eagle:library:325" package="1X02" package3d_urn="urn:adsk.eagle:package:22435/2" value="" x="-67.31" y="-87.63"/>
+<element name="C2" library="rcl" library_urn="urn:adsk.eagle:library:334" package="C0603" value=".1uF" x="-73.66" y="-97.79"/>
+<element name="C3" library="rcl" library_urn="urn:adsk.eagle:library:334" package="E2,5-6E" value="10uF" x="-66.04" y="-109.22"/>
+<element name="C4" library="rcl" library_urn="urn:adsk.eagle:library:334" package="C0603" value=".1uF" x="-73.66" y="-120.65"/>
 </elements>
 <signals>
@@
 <contactref element="SW2" pad="D"/>
 <contactref element="SW2" pad="C"/>
+<contactref element="JP1" pad="1"/>
+<contactref element="C2" pad="1"/>
+<contactref element="C3" pad="-"/>
+<contactref element="C4" pad="1"/>
+<wire x1="-64.77" y1="-109.22" x2="-74.51" y2="-120.65" width="0" layer="19" extent="1-1"/>
+<wire x1="-74.51" y1="-97.79" x2="-64.77" y2="-109.22" width="0" layer="19" extent="1-1"/>
+<wire x1="-68.58" y1="-87.63" x2="-74.51" y2="-97.79" width="0" layer="19" extent="1-1"/>
+<wire x1="-53.34" y1="-65.92" x2="-68.58" y2="-87.63" width="0" layer="19" extent="1-1"/>
 <wire x1="-55.84" y1="-51.42" x2="-53.34" y2="-65.92" width="0" layer="19" extent="1-1"/>
 <wire x1="-63.5" y1="-13.97" x2="-55.84" y2="-51.42" width="0" layer="19" extent="1-1"/>
@@
 <contactref element="R9" pad="2"/>
 <contactref element="R10" pad="2"/>
-<wire x1="-33.02" y1="67.31" x2="-20.74" y2="80.01" width="0" layer="19" extent="1-1"/>
-<wire x1="-43.6" y1="68.58" x2="-33.02" y2="67.31" width="0" layer="19" extent="1-1"/>
+<contactref element="JP1" pad="2"/>
+<wire x1="-43.6" y1="68.58" x2="-66.04" y2="-87.63" width="0" layer="19" extent="1-1"/>
+<wire x1="-33.02" y1="67.31" x2="-43.6" y2="68.58" width="0" layer="19" extent="1-1"/>
 <wire x1="-44.87" y1="85.09" x2="-43.6" y2="68.58" width="0" layer="19" extent="1-1"/>
+<wire x1="-20.74" y1="80.01" x2="-33.02" y2="67.31" width="0" layer="19" extent="1-1"/>
 </signal>
 <signal name="WAKE">
@@
 <contactref element="R3" pad="2"/>
 <contactref element="R4" pad="2"/>
-<wire x1="-69" y1="-77.47" x2="-74.08" y2="-77.47" width="0" layer="19" extent="1-1"/>
+<contactref element="C4" pad="2"/>
+<contactref element="C3" pad="+"/>
+<wire x1="-67.31" y1="-109.22" x2="-72.81" y2="-120.65" width="0" layer="19" extent="1-1"/>
+<wire x1="-69" y1="-77.47" x2="-67.31" y2="-109.22" width="0" layer="19" extent="1-1"/>
+<wire x1="-74.08" y1="-77.47" x2="-69" y2="-77.47" width="0" layer="19" extent="1-1"/>
 <wire x1="-63.92" y1="-77.47" x2="-69" y2="-77.47" width="0" layer="19" extent="1-1"/>
 <wire x1="-49.53" y1="55.22" x2="-63.92" y2="-77.47" width="0" layer="19" extent="1-1"/>
@@
 <contactref element="C1" pad="+"/>
 <contactref element="JP6" pad="1"/>
-<wire x1="-20.32" y1="62.23" x2="-68.58" y2="-34.29" width="0" layer="19" extent="1-1"/>
+<contactref element="C2" pad="2"/>
+<contactref element="IC1" pad="3"/>
+<wire x1="-68.58" y1="-34.29" x2="-72.81" y2="-97.79" width="0" layer="19" extent="1-1"/>
+<wire x1="-47.23" y1="48.92" x2="-68.58" y2="-34.29" width="0" layer="19" extent="1-1"/>
+<wire x1="-20.32" y1="62.23" x2="-47.23" y2="48.92" width="0" layer="19" extent="1-1"/>
 </signal>
 <signal name="PWM_CONTROL">
@@
 </signal>
 <signal name="N$24">
+<contactref element="IC3" pad="12"/>
 <contactref element="R22" pad="2"/>
-<contactref element="IC3" pad="12"/>
 <wire x1="-21.38" y1="49.09" x2="-20.74" y2="74.93" width="0" layer="19" extent="1-1"/>
 </signal>
